File: Player.sch (EAGLE design)
At the start: 60 parts, among them CN1 STEREO-3.5-MJ8435, CON1 UART-S, CON2 MICROSD-DM3, CON3 MINI-USB-, CON4 MOLEX-5251-02-S_LONG, IC1 R5F5631-48LFQFP, IC2 AK4386, IC3 BH3544F, IC4 XC6802A42XMR, IC6 AQM1248-RN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

Commit message: Halfway through wiring
Parts:
- removed C15: 0.1u, Passive_Robotech:C-2012
- removed D1: RB160M-30TR, Diode_Robotech:DIODE-SMD3216
- removed SW7: SLIDESW, Passive_Robotech:SLIDESW
- added C30: 22u, Passive_Robotech:CC-2.5-8
- added Q1: SSM6L35FE, Transistor_Robotech:SSM6L35FE
- added R10, R11: 100, Passive_Robotech:R-2012
- added R12: 10k, Passive_Robotech:R-2012
- added R13, R14: 22k, Passive_Robotech:R-2012
- C19, C20, C23: device Passive_Robotech:CC-2.5-7 -> Passive_Robotech:CC-2.5-8
Connections:
- new net N$55: IC1.P46, R13.2, R14.2
- net +3V3: now also IC1.VCC_USB; no longer C22.1, IC3.VCC
- net +5V: now also C22.1, C26.1, C30.+, IC3.VCC, Q1P.S, R12.1, R13.1, U$1.CONTROL, U$1.VIN; no longer D1.C, SW7.O
- net GND: now also C30.-, Q1N.S, R14.1; no longer C15.2
- net N$18: now also IC1.PE2, R10.2; no longer C15.1, IC1.VCC_USB
- net N$19: now also Q1N.G, R10.1; no longer CON3.2, IC1.USB0_DM
- net N$21: now also Q1P.G, R11.1, R12.2; no longer CON3.3, IC1.USB0_DP
- net N$47: now also Q1N.D, R11.2; no longer C26.1, SW7.P, U$1.CONTROL, U$1.VIN
- net N$50: now also Q1P.D; no longer D1.A
- net N$54: now also IC1.PB0; no longer IC1.PE2
Other:
- moved on the sheet: CN1, R9
